File: TwomesGateway/TwomesGateway.kicad_pcb (KiCad board)
At the start: 2 copper layers, 35.6 x 79 mm, 36 parts, among them J1 FTDI header, J2 RJ12-6P6C, J3 USB_B_Micro, J4 Conn_01x06, M3 MountingHole_3.2mm_M3, Q1 BC807, Q2 BC807, Q3 BC807, Q4 MMBT3904, SW1 SW_Push, SW2 SW_Push, SW3 SW_Push, U1 AP7365-33WG-7, U2 ESP32-WROOM-32D

Commit message: Add files via upload
Parts:
- removed REF**: OSHW-Logo2_9.8x8mm_SilkScreen, Symbol:OSHW-Logo2_9.8x8mm_SilkScreen
